Commit message: added apriltag to office and added camera to robot

File: rse_gazebo/urdf/rse_bot.urdf.xacro (robot description, xacro)
@@ -39,4 +39,23 @@
     </visual>
   </link>
+  <link name="camera_link">
+    <visual>
+      <geometry>
+        <box size="0.04 0.06 0.04"/>
+      </geometry>
+    </visual>
+  </link>
+  <joint name="camera_joint" type="fixed">
+    <parent link="base_link"/>
+    <child link="camera_link"/>
+    <origin xyz="0.19 0 0.10" rpy="0 0 0"/>
+  </joint>
+  <link name="camera_optical_frame"/>
+  <joint name="camera_optical_joint" type="fixed">
+    <parent link="camera_link"/>
+    <child link="camera_optical_frame"/>
+    <origin xyz="0 0 0"
+            rpy="-1.57079632679 0 -1.57079632679"/>
+  </joint>
   <joint name="right_wheel_joint" type="continuous">
     <parent link="base_link"/>
